File: PCB/Hackpad.kicad_sch (KiCad schematic)
At the start: 40 parts, among them J1 Conn_01x04, SW1 SW_Push, SW2 SW_Push, SW3 SW_Push, SW4 SW_Push, SW5 SW_Push, SW6 SW_Push, SW7 SW_Push, SW8 SW_Push, SW9 RotaryEncoder_Switch, U1 MOUDLE-SEEEDUINO-XIAO

Commit message: Modified Schematics
Other:
- note removed: "3 Modes: 1. Jog wheel 2. Volume 3. Music picker via rotating"
- company: (none) -> Lix
- title: (none) -> Mediapad
Changed lines of the file:
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@@
 	(generator_version "10.0")
 	(paper "A4")
+	(title_block
+		(title "Mediapad")
+		(date "2026-07-23")
+		(rev "1.0")
+		(company "Lix")
+		(comment 1 "it is a part of the Hackpad mission/project.")
+		(comment 2 "This schematic is for Mediapad, created by Lix and")
+	)
 	(text "SDA"
 		(exclude_from_sim no)
@@
 		(effects
 			(font
-				(size 1.27 1.27)
-			)
-		)
-	)
-	(text "3 Modes:\n	1. Jog wheel\n	2. Volume\n	3. Music picker via rotating"
-		(exclude_from_sim no)
-		(at 304.546 117.602 0)
-		(effects
-			(font
